Commit message: rviz launch works

File: urdf/BASE_ROBOT.urdf.xacro (robot description, xacro)
@@ -4,5 +4,5 @@
      Commit Version: 1.6.0-4-g7f85cfe  Build Version: 1.6.7995.38578
      For more information, please see http://wiki.ros.org/sw_urdf_exporter -->
-<robot xmlns:xacro="http://ros.org/wiki/xacro"  name="BASE_ROBOT">
+<robot xmlns:xacro="http://ros.org/wiki/xacro" name="BASE_ROBOT">
   <xacro:include filename="$(find robot_description)/urdf/BASE_ROBOT_ESSENTIALS.xacro" />
   <xacro:include filename="$(find robot_description)/urdf/gazebo_essentials_base.xacro" />
@@ -19,5 +19,5 @@
         rpy="0 0 0" />
       <mass
-        value="0.16211" />
+        value=".16211" />
       <inertia
         ixx="0.0001472"

File: urdf/gazebo_essentials_base.xacro (robot description, xacro)
@@ -23,5 +23,5 @@
         <commandTopic>cmd_vel</commandTopic>
         <odometryTopic>odom</odometryTopic>
-        <robotBaseFrame>base_link</robotBaseFrame>
+        <robotBaseFrame>dummy</robotBaseFrame>
         <wheelAcceleration>2.8</wheelAcceleration>
         <publishWheelJointState>true</publishWheelJointState>
@@ -43,12 +43,18 @@
 <xacro:macro name="wheel_friction" params="prefix ">
 <gazebo reference="${prefix}_LINK">
+  <material>
+    Gazebo/Blue
+  </material>
  <mu1 value="1.0"/>
  <mu2 value="1.0"/>
- <kp value="10000000.0" />
- <kd value="1.0" />
- <fdir1 value="1 0 0"/>
+ <fdir value="1 0 0"/>
  <turnGravityOff>false</turnGravityOff>
 </gazebo>
 </xacro:macro>
 <!--######################################################################-->
+<gazebo reference="base_link">
+  <material>
+    Gazebo/Red
+  </material>
+</gazebo>
 </robot>
